File: Original_NES/CPU.sch (KiCad schematic (older format))
At the start: 27 parts, among them Q2 2SC2021, Q3 2SC2021, U6 RP2A03, X1 21.47727MHz

Commit message: Finish Clock Generator
Connections:
- net labels added: CPU_CLK, PPU_PIN_13
- net labels removed: CLK
- wire segments 42 -> 44
Other:
- moved on the sheet: R13
Changed lines of the file:
@@
 Text GLabel 3600 2200 0    50   Input ~ 0
 ~RESET~
-Text GLabel 2650 2400 0    50   Input ~ 0
-CLK
+Text GLabel 1700 6450 1    50   Output ~ 0
+CPU_CLK
 Text GLabel 3600 3300 0    50   Output ~ 0
 RW
@@
 L Device:R R13
 U 1 1 5ED2B253
-P 2000 6550
-F 0 "R13" V 2100 6550 50  0000 C CNN
-F 1 "150k" V 2000 6550 50  0000 C CNN
-F 2 "" V 1930 6550 50  0001 C CNN
-F 3 "~" H 2000 6550 50  0001 C CNN
-	1    2000 6550
+P 1700 6850
+F 0 "R13" V 1800 6850 50  0000 C CNN
+F 1 "150k" V 1700 6850 50  0000 C CNN
+F 2 "" V 1630 6850 50  0001 C CNN
+F 3 "~" H 1700 6850 50  0001 C CNN
+	1    1700 6850
 	-1   0    0    1
 $EndComp
@@
 	1    0    0    -1
 $EndComp
+Text GLabel 4400 5900 2    50   Output ~ 0
+PPU_PIN_13
+$Comp
+L power:GND #PWR?
+U 1 1 5ED5879E
+P 1700 7000
+F 0 "#PWR?" H 1700 6750 50  0001 C CNN
+F 1 "GND" H 1705 6827 50  0000 C CNN
+F 2 "" H 1700 7000 50  0001 C CNN
+F 3 "" H 1700 7000 50  0001 C CNN
+	1    1700 7000
+	1    0    0    -1
+$EndComp
+Wire Wire Line
+	2000 6700 1700 6700
+Text GLabel 3600 2400 0    50   Input ~ 0
+CPU_CLK
+Wire Wire Line
+	1700 6700 1700 6450
+Connection ~ 1700 6700
 $EndSCHEMATC

Commit message: Add more things
Parts:
- removed C? (x2): 330pF, symbol Device:C
- removed R? (x2): 20k, symbol Device:R
- removed R?: 12k, symbol Device:R
- removed R? (x2): 5.6k, symbol Device:R
- added BOTTOM: AUX PORT, symbol Connector_Generic:Conn_02x24_Counter_Clockwise
- added C10, C24, C39: 0.01uF, symbol Device:C
- added EDGE: CARTRIDGE, symbol Connector_Generic:Conn_02x36_Counter_Clockwise
- added J?: For Reference Only. Pin numbering doesn't match b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, symbol Connector_Generic:Conn_02x36_Top_Bottom
- added U2: 74LS373, symbol 74xx:74LS373
- added U3: 74LS139, symbol 74xx:74LS139
- added U5: RP2C02, Package_DIP:DIP-40_W15.24mm, symbol _NTSCustom:RP2C02
Connections:
- net labels added: PPU_A13, PPU_CLK, ~OE1, ~OE2
- net labels removed: AUDIO, EXP_7, OE1, OE2, PPU_PIN_13
- wire segments 44 -> 31
- no-connect marks 0 -> 4
Other:
- note added: "Clock Generator\n"
- moved on the sheet: C13, C25, C32, C41, C42, C43, C44, C45, C?, Q2, Q3, R10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

Commit message: Add RAM and stuff
Parts:
- added C22, C3, C46: 0.01uF, symbol Device:C
- added U1, U4: TMM2115, Package_DIP:DIP-24_W7.62mm, symbol _NTSCustom:TMM2115
Connections:
- net labels added: CPU_M2, CPU_NMI, CPU_RAM_CS, CPU_RW, Cartridge22, Cartridge52, Cartridge59, PPU_A0, PPU_A1, PPU_A10, PPU_A11, PPU_A12, PPU_A2, PPU_A3, PPU_A4, PPU_A5, PPU_A6, PPU_A7, PPU_A8, PPU_A9, PPU_AD0, PPU_AD1, PPU_AD2, PPU_AD3, PPU_AD4, PPU_AD5, PPU_AD6, PPU_AD7, PPU_ALE, PPU_CS, PPU_RD, PPU_WR
- net labels removed: IRQ, M2, NMI, OUT0, OUT1, OUT2, RW, ~OE1, ~OE2, ~RESET~
Other:
- moved on the sheet: C10, C39, C41, C42, C43, C44, C45, C?, Q2, Q3, R10, R11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
