File: Original_NES/Original_NES.sch (KiCad schematic (older format))
At the start: 0 parts

Commit message: Delete extra files
Parts:
- added AUX1: AUX PORT, symbol Connector_Generic:Conn_02x24_Counter_Clockwise
- added BC1, BC2, C8: 0.1uF, symbol Device:C
- added C1: 100uF, symbol Device:CP
- added C10, C11, C12, C13, C14, C15, C16, C17, C18, C19, C22, C24, C25, C3, C32, C39, C4, C40, C46: 0.01uF, symbol Device:C
- added C2: 1N4148?, symbol Device:D
- added C20, C21, C44, C6, C7: 220pF, symbol Device:C
- added C23: 1uF, symbol Device:CP
- added C27, C28, C29, C30, C31, C33, C34, C35, C36, C37, C5: 330pF, symbol Device:C
- added C41: 18pF, symbol Device:C
- added C42: 15pF, symbol Device:C
- added C43, C45: 51pF, symbol Device:C
- added C9: 2.2uF, symbol Device:CP
- added DA1, DA3: DAN601, symbol _NTSCustom:DAN601
- added DA2, DA4: uPA64H, symbol _NTSCustom:uPA64H
- added EDGE1: CARTRIDGE, symbol Connector_Generic:Conn_02x36_Counter_Clockwise
- added FC1: 39uH, symbol Device:L
- added FC2: ?uH, symbol Device:Ferrite_Bead
- added P4: P1 PAD, symbol Connector:Conn_01x07_Male
- added P5: P2 PAD, symbol Connector:Conn_01x07_Male
- added P6: Power/Reset, symbol Connector:Conn_01x05_Male
- added Q1: 2SA937, symbol Device:Q_PNP_ECB
- added Q2, Q3: 2SC2021, symbol Device:Q_NPN_BCE
- added R1: 1M, symbol Device:R
- added R10: 220k, symbol Device:R
- added R11, R12, R2: 510, symbol Device:R
- added R13: 150k, symbol Device:R
- added R14, R15: 5.6k, symbol Device:R
- added R16: 10k, symbol Device:R
- added R3, R4: 100, symbol Device:R
- added R5: 220, symbol Device:R
- added R6: 47K, symbol Device:R
- added R7, R9: 20K, symbol Device:R
- added R8: 12K, symbol Device:R
- added RA1: 12x 10k, Resistor_THT:R_Array_SIP13, symbol Device:R_Network12
- added RA2: 6.8k, Resistor_THT:R_Array_SIP5, symbol Device:R_Network04
- added REFERENCE1: For Reference Only. Pin numbering doesn't match b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, symbol Connector_Generic:Conn_02x36_Top_Bottom
- added RF_MOD1: RF MOD, symbol Connector:Conn_01x05_Male
- added TC1: 30pF, symbol Device:CTRIM
- added U1, U4: TMM2115, Package_DIP:DIP-24_W7.62mm, symbol _NTSCustom:TMM2115
- added U10: 3193A, Package_DIP:DIP-16_W7.62mm, symbol _NTSCustom:3193A
- added U2: 74LS373, symbol 74xx:74LS373
- added U3: 74LS139, symbol 74xx:74LS139
- added U5: RP2C02, Package_DIP:DIP-40_W15.24mm, symbol _NTSCustom:RP2C02
- added U6: RP2A03, Package_DIP:DIP-40_W15.24mm, symbol _NTSCustom:RP2A03
- added U7, U8: 74LS368, symbol 74xx:74LS368
- added U9: 74HC04, symbol 74xx:74HC04
- added X1: 21.47727MHz, symbol Device:Crystal
- added X2: 4MHz, symbol Device:Resonator
Connections:
- new net: R4.1, R7.1, U6.1 (AD1)
- new net: R3.1, R8.1, U6.2 (AD2)
- new net: C42.2, C45.1, Q2.2 (C), Q3.1 (B), R10.1, R11.1, X1.1
- new net: C41.1, TC1.2, X1.2
- new net: C41.2, C43.2, Q2.1 (B), R10.2, TC1.1
- new net: Q1.3 (B), U5.21 (VOUT)
- new net: C7.1, R1.1, U9.1, X2.3
- new net: C6.1, R1.2, U9.13, U9.2, U9.3, X2.1
- new net: R5.1, U9.8
- new net: C21.2, C23.1, R6.1, U9.11
- new net: U10.6 (CLK), U9.12
- new net: U3.1 (E), U3.11 (O1)
- new net: C9.2, U10.3 (R02)
- new net: C23.2, R7.2, R8.2, R9.1
- new net +5V: AUX1.1 (Pin_1), AUX1.48 (Pin_48), BC1.1, BC2.1, C1.1, C10.1, C13.1, C16.1, C19.1, C22.1, C24.1, C25.1, C3.1, C32.1, C39.1, C40.1, C46.1, C8.1, C9.1, DA1.4, DA2.7, DA3.4, DA4.1, EDGE1.36 (Pin_36), P4.5 (Pin_5), P5.5 (Pin_5), P6.3 (Pin_3), Q3.2 (C), R11.2, R14.1, R15.1, R16.1, R2.2, RA1.1 (common), RA2.1 (common), REFERENCE1.36 (Pin_36), RF_MOD1.3 (Pin_3), U1.24 (+5V), U10.16 (VCC), U10.4 (SEL), U2.20 (VCC), U3.16 (VCC), U4.24 (+5V), U5.40 (+5V), U6.40 (+5V), U7.16 (VCC), U8.16 (VCC), U9.14 (VCC)
- new net AUDIO_OUT: C4.1, FC1.1, RF_MOD1.2 (Pin_2)
- new net AUX_AUDIO_IN: AUX1.3 (Pin_3), R9.2
- new net AUX_AUDIO_OUT: AUX1.22 (Pin_22), C20.1, C21.1, FC1.2, R6.2, U9.10
- new net AUX_VIDEO_OUT: AUX1.21 (Pin_21), FC2.1, Q1.1 (E), R2.1
- new net CART_CLK: C44.1, EDGE1.72 (Pin_72), Q3.3 (E), R12.2, REFERENCE1.37 (Pin_37)
- new net CIC_CLK: AUX1.24 (Pin_24), EDGE1.38 (Pin_38), REFERENCE1.71 (Pin_71), U9.4
- new net CIC_IN: C2.1 (K), EDGE1.35 (Pin_35), REFERENCE1.35 (Pin_35), U10.2 (IN)
- new net CIC_OUT: EDGE1.34 (Pin_34), REFERENCE1.34 (Pin_34), U10.1 (OUT)
- new net CIC_RST: EDGE1.39 (Pin_39), REFERENCE1.70 (Pin_70), U10.10 (R11)
- new net CIRAM_A10: EDGE1.22 (Pin_22), REFERENCE1.22 (Pin_22), U4.19 (A10)
- new net CIRAM_CE: EDGE1.52 (Pin_52), REFERENCE1.57 (Pin_57), U4.18 (~CE)
- new net CPU_A0: EDGE1.13 (Pin_13), REFERENCE1.13 (Pin_13), U1.8 (A0), U5.12 (CPU_A0), U6.4 (A0)
- new net CPU_A1: EDGE1.12 (Pin_12), REFERENCE1.12 (Pin_12), U1.7 (A1), U5.11 (CPU_A1), U6.5 (A1)
- new net CPU_A10: EDGE1.3 (Pin_3), REFERENCE1.3 (Pin_3), U1.19 (A10), U6.14 (A10)
- new net CPU_A11: EDGE1.2 (Pin_2), REFERENCE1.2 (Pin_2), U6.15 (A11)
- new net CPU_A12: EDGE1.70 (Pin_70), REFERENCE1.39 (Pin_39), U6.16 (A12)
- new net CPU_A13: EDGE1.69 (Pin_69), REFERENCE1.40 (Pin_40), U3.2 (A0), U6.17 (A13)
- new net CPU_A14: EDGE1.68 (Pin_68), REFERENCE1.41 (Pin_41), U3.3 (A1), U6.18 (A14)
- new net CPU_A15: AUX1.5 (Pin_5), U3.13 (A1), U6.19 (A15)
- new net CPU_A2: EDGE1.11 (Pin_11), REFERENCE1.11 (Pin_11), U1.6 (A2), U5.10 (CPU_A2), U6.6 (A2)
- new net CPU_A3: EDGE1.10 (Pin_10), REFERENCE1.10 (Pin_10), U1.5 (A3), U6.7 (A3)
- new net CPU_A4: EDGE1.9 (Pin_9), REFERENCE1.9 (Pin_9), U1.4 (A4), U6.8 (A4)
- new net CPU_A5: EDGE1.8 (Pin_8), REFERENCE1.8 (Pin_8), U1.3 (A5), U6.9 (A5)
- new net CPU_A6: EDGE1.7 (Pin_7), REFERENCE1.7 (Pin_7), U1.2 (A6), U6.10 (A6)
- new net CPU_A7: EDGE1.6 (Pin_6), REFERENCE1.6 (Pin_6), U1.1 (A7), U6.11 (A7)
- new net CPU_A8: EDGE1.5 (Pin_5), REFERENCE1.5 (Pin_5), U1.23 (A8), U6.12 (A8)
- new net CPU_A9: EDGE1.4 (Pin_4), REFERENCE1.4 (Pin_4), U1.22 (A9), U6.13 (A9)
- new net CPU_CLK: C44.2, R13.2, U6.29 (CLK)
- new net CPU_D0: AUX1.32 (Pin_32), EDGE1.60 (Pin_60), REFERENCE1.49 (Pin_49), U1.9 (D0), U5.2 (CPU_D0), U6.28 (D0), U7.3 (O1a), U8.3 (O1a)
- new net CPU_D1: AUX1.31 (Pin_31), EDGE1.61 (Pin_61), REFERENCE1.48 (Pin_48), U1.10 (D1), U5.3 (CPU_D1), U6.27 (D1), U7.5 (O2a), U8.5 (O2a)
- new net CPU_D2: AUX1.30 (Pin_30), EDGE1.62 (Pin_62), REFERENCE1.47 (Pin_47), U1.11 (D2), U5.4 (CPU_D2), U6.26 (D2), U7.9 (O4a), U8.9 (O4a)
- new net CPU_D3: AUX1.29 (Pin_29), EDGE1.63 (Pin_63), REFERENCE1.46 (Pin_46), U1.13 (D3), U5.5 (CPU_D3), U6.25 (D3), U7.11 (O5b), U8.11 (O5b)
- new net CPU_D4: AUX1.28 (Pin_28), EDGE1.64 (Pin_64), REFERENCE1.45 (Pin_45), U1.14 (D4), U5.6 (CPU_D4), U6.24 (D4), U7.13 (O6b), U8.13 (O6b)
- new net CPU_D5: AUX1.27 (Pin_27), EDGE1.65 (Pin_65), REFERENCE1.44 (Pin_44), U1.15 (D5), U5.7 (CPU_D5), U6.23 (D5)
- new net CPU_D6: AUX1.26 (Pin_26), EDGE1.66 (Pin_66), REFERENCE1.43 (Pin_43), U1.16 (D6), U5.8 (CPU_D6), U6.22 (D6)
- new net CPU_D7: AUX1.25 (Pin_25), EDGE1.67 (Pin_67), REFERENCE1.42 (Pin_42), U1.17 (D7), U5.9 (CPU_D7), U6.21 (D7)
- new net CPU_IRQ: AUX1.14 (Pin_14), EDGE1.15 (Pin_15), RA1.7 (R6), REFERENCE1.15 (Pin_15), U6.32 (~IRQ~)
- new net CPU_M2: EDGE1.71 (Pin_71), REFERENCE1.38 (Pin_38), U3.14 (A0), U6.31 (M2)
- new net CPU_NMI: AUX1.4 (Pin_4), R16.2, RA1.13 (R12), U5.19 (~INT), U6.33 (~NMI~)
- new net CPU_OE1: AUX1.34 (Pin_34), AUX1.37 (Pin_37), C33.1, DA1.1, DA2.1, P4.2 (Pin_2), R15.2, RA2.4 (R3), U6.36 (~OE1~), U7.1 (OEa), U7.15 (OEb)
- new net CPU_OE2: AUX1.11 (Pin_11), AUX1.17 (Pin_17), C27.1, DA3.2, DA4.2, P5.2 (Pin_2), R14.2, RA2.5 (R4), U6.35 (~OE2~), U8.1 (OEa), U8.15 (OEb)
- new net CPU_OUT0: AUX1.43 (Pin_43), C28.1, C34.1, DA1.2, DA2.2, DA3.3, DA4.3, P4.3 (Pin_3), P5.3 (Pin_3), RA2.2 (R1), U6.39 (OUT0)
- new net CPU_OUT1: AUX1.44 (Pin_44), U6.38 (OUT1)
- new net CPU_OUT2: AUX1.45 (Pin_45), U6.37 (OUT2)
- new net CPU_RAM_CS: U1.18 (~CE), U3.4 (O0)
- new net CPU_RST: U10.9 (R10), U5.22 (~RST), U6.3 (~RESET~), U9.9
- new net CPU_RW: EDGE1.14 (Pin_14), REFERENCE1.14 (Pin_14), U1.21 (~WE), U5.1 (R/W), U6.34 (R/W)
- new net EXP0: AUX1.42 (Pin_42), EDGE1.16 (Pin_16), REFERENCE1.16 (Pin_16)
- new net EXP1: AUX1.41 (Pin_41), EDGE1.17 (Pin_17), REFERENCE1.17 (Pin_17)
- new net EXP2: AUX1.40 (Pin_40), EDGE1.18 (Pin_18), REFERENCE1.18 (Pin_18)
- new net EXP3: AUX1.39 (Pin_39), EDGE1.19 (Pin_19), REFERENCE1.19 (Pin_19)
- new net EXP4: AUX1.38 (Pin_38), EDGE1.20 (Pin_20), REFERENCE1.20 (Pin_20)
- new net EXP5: AUX1.10 (Pin_10), EDGE1.54 (Pin_54), REFERENCE1.55 (Pin_55)
- new net EXP6: AUX1.9 (Pin_9), EDGE1.55 (Pin_55), REFERENCE1.54 (Pin_54)
- new net EXP7: AUX1.8 (Pin_8), EDGE1.56 (Pin_56), REFERENCE1.53 (Pin_53)
- new net EXP8: AUX1.7 (Pin_7), EDGE1.57 (Pin_57), REFERENCE1.52 (Pin_52)
- new net EXP9: AUX1.6 (Pin_6), EDGE1.58 (Pin_58), REFERENCE1.51 (Pin_51)
- new net GND: AUX1.2 (Pin_2), AUX1.47 (Pin_47), BC1.2, BC2.2, C1.2, C10.2, C11.2, C12.2, C13.2, C14.2, C15.2, C16.2, C17.2, C18.2, C19.2, C2.2 (A), C20.2, C22.2, C24.2, C25.2, C27.2, C28.2, C29.2, C3.2, C30.2, C31.2, C32.2, C33.2, C34.2, C35.2, C36.2, C37.2, C39.2, C4.2, C40.2, C42.1, C43.1, C46.2, C5.2, C6.2, C7.2, DA1.7, DA2.4, DA3.1, DA4.4, EDGE1.1 (Pin_1), EDGE1.37 (Pin_37), P4.1 (Pin_1), P5.1 (Pin_1), Q1.2 (C), Q2.3 (E), R12.1, R13.1, R3.2, R4.2, REFERENCE1.1 (Pin_1), REFERENCE1.72 (Pin_72), U1.12 (GND), U1.20 (~OE), U10.11 (R12), U10.12 (R13), U10.13 (R20), U10.14 (R21), U10.15 (R22), U10.8 (GND), U2.1 (OE), U2.10 (GND), U3.15 (E), U3.8 (GND), U4.12 (GND), U5.14 (EXT0), U5.15 (EXT1), U5.16 (EXT2), U5.17 (EXT3), U5.20 (GND), U6.20 (GND), U6.30 (TST), U7.6 (I3), U7.8 (GND), U8.6 (I3), U8.8 (GND), U9.7 (GND), X2.2
- new net P1_D0: AUX1.35 (Pin_35), C35.1, DA1.3, DA2.3, DA3.5, DA4.5, P4.4 (Pin_4), RA1.9 (R8), U7.2 (I1)
- new net P1_D1: AUX1.12 (Pin_12), AUX1.20 (Pin_20), RA1.8 (R7), U7.4 (I2)
- new net P1_D2: AUX1.33 (Pin_33), RA1.12 (R11), U7.10 (I4)
- new net P1_D3: AUX1.13 (Pin_13), C36.1, DA1.5, DA2.5, DA3.6, DA4.6, P4.6 (Pin_6), RA1.10 (R9), U7.12 (I5)
- new net P1_D4: AUX1.36 (Pin_36), C37.1, DA1.6, DA2.6, DA3.7, DA4.7, P4.7 (Pin_7), RA1.11 (R10), U7.14 (I6)
- new net P2_D0: AUX1.19 (Pin_19), C29.1, P5.4 (Pin_4), RA1.3 (R2), U8.2 (I1)
- new net P2_D1: RA1.2 (R1), U8.4 (I2)
- new net P2_D2: AUX1.15 (Pin_15), RA1.6 (R5), U8.10 (I4)
- new net P2_D3: AUX1.16 (Pin_16), C30.1, P5.6 (Pin_6), RA1.5 (R4), U8.12 (I5)
- new net P2_D4: AUX1.18 (Pin_18), C31.1, P5.7 (Pin_7), RA1.4 (R3), U8.14 (I6)
- new net PPU_!A13: EDGE1.51 (Pin_51), REFERENCE1.58 (Pin_58), U9.6
- new net PPU_A0: EDGE1.29 (Pin_29), REFERENCE1.29 (Pin_29), U2.9 (O3), U4.8 (A0)
- new net PPU_A1: EDGE1.28 (Pin_28), REFERENCE1.28 (Pin_28), U2.12 (O4), U4.7 (A1)
- new net PPU_A10: EDGE1.46 (Pin_46), REFERENCE1.63 (Pin_63), U5.28 (PPU_A10)
- new net PPU_A11: EDGE1.47 (Pin_47), REFERENCE1.62 (Pin_62), U5.27 (PPU_A11)
- new net PPU_A12: EDGE1.45 (Pin_45), REFERENCE1.64 (Pin_64), U5.26 (PPU_A12)
- new net PPU_A13: EDGE1.44 (Pin_44), RA2.3 (R2), REFERENCE1.65 (Pin_65), U5.25 (PPU_A13), U9.5
- new net PPU_A2: EDGE1.27 (Pin_27), REFERENCE1.27 (Pin_27), U2.6 (O2), U4.6 (A2)
- new net PPU_A3: EDGE1.26 (Pin_26), REFERENCE1.26 (Pin_26), U2.15 (O5), U4.5 (A3)
- new net PPU_A4: EDGE1.25 (Pin_25), REFERENCE1.25 (Pin_25), U2.5 (O1), U4.4 (A4)
- new net PPU_A5: EDGE1.24 (Pin_24), REFERENCE1.24 (Pin_24), U2.16 (O6), U4.3 (A5)
- new net PPU_A6: EDGE1.23 (Pin_23), REFERENCE1.23 (Pin_23), U2.2 (O0), U4.2 (A6)
- new net PPU_A7: EDGE1.50 (Pin_50), REFERENCE1.59 (Pin_59), U2.19 (O7), U4.1 (A7)
- new net PPU_A8: EDGE1.49 (Pin_49), REFERENCE1.60 (Pin_60), U4.23 (A8), U5.30 (PPU_A8)
- new net PPU_A9: EDGE1.48 (Pin_48), REFERENCE1.61 (Pin_61), U4.22 (A9), U5.29 (PPU_A9)
- new net PPU_AD0: EDGE1.30 (Pin_30), REFERENCE1.30 (Pin_30), U2.8 (D3), U4.9 (D0), U5.38 (PPU_AD0)
- new net PPU_AD1: EDGE1.31 (Pin_31), REFERENCE1.31 (Pin_31), U2.13 (D4), U4.10 (D1), U5.37 (PPU_AD1)
- new net PPU_AD2: EDGE1.32 (Pin_32), REFERENCE1.32 (Pin_32), U2.7 (D2), U4.11 (D2), U5.36 (PPU_AD2)
- new net PPU_AD3: EDGE1.33 (Pin_33), REFERENCE1.33 (Pin_33), U2.14 (D5), U4.13 (D3), U5.35 (PPU_AD3)
- new net PPU_AD4: EDGE1.40 (Pin_40), REFERENCE1.69 (Pin_69), U2.4 (D1), U4.14 (D4), U5.34 (PPU_AD4)
- new net PPU_AD5: EDGE1.41 (Pin_41), REFERENCE1.68 (Pin_68), U2.17 (D6), U4.15 (D5), U5.33 (PPU_AD5)
- new net PPU_AD6: EDGE1.42 (Pin_42), REFERENCE1.67 (Pin_67), U2.3 (D0), U4.16 (D6), U5.32 (PPU_AD6)
- new net PPU_AD7: EDGE1.43 (Pin_43), REFERENCE1.66 (Pin_66), U2.18 (D7), U4.17 (D7), U5.31 (PPU_AD7)
- new net PPU_ALE: U2.11 (LE), U5.39 (ALE)
- new net PPU_CLK: C45.2, U5.18 (CLK)
- new net PPU_CS: U3.5 (O1), U5.13 (~CS)
- new net PPU_RD: EDGE1.21 (Pin_21), REFERENCE1.21 (Pin_21), U4.20 (~OE), U5.24 (~RD)
- new net PPU_WR: EDGE1.53 (Pin_53), REFERENCE1.56 (Pin_56), U4.21 (~WE), U5.23 (~WR)
- new net PWR_LED: C18.1, P6.5 (Pin_5), R5.2
- new net PWR_SW_IN: C11.1, C14.1, P6.1 (Pin_1), RF_MOD1.5 (Pin_5)
- new net PWR_SW_OUT: AUX1.23 (Pin_23), C12.1, C15.1, P6.2 (Pin_2), RF_MOD1.4 (Pin_4)
- new net ROMSEL: EDGE1.59 (Pin_59), REFERENCE1.50 (Pin_50), U3.9 (O3)
- new net RST_PB: C17.1, C8.2, P6.4 (Pin_4), U10.7 (RST)
- new net VIDEO_OUT: C5.1, FC2.2, RF_MOD1.1 (Pin_1)
- no-connect marks 0 -> 8
Other:
- note added: "C6 and C7\nnot populated\n"
- note added: "CIC\n"
- note added: "Clock Generator\n"
- note added: "Controller Inputs\n"
- note added: "Power/Reset Connector\n"
- note added: "R14, R15, and R16\nnot populated\n"
