File: HVC-001 Console/HVC-001.sch (KiCad schematic (older format))
At the start: 93 parts, among them P4 P1 PAD, P5 P2 PAD, P6 Power/Reset, Q1 2SA937, Q2 2SC2021, Q3 2SC2021, U1 TMM2115, U10 3193A, U2 74LS373, U3 74LS139, U4 TMM2115, U5 RP2C02, U6 RP2A03, U7 74LS368, U8 74LS368, U9 74HC04, X1 21.47727MHz, X2 4MHz

Commit message: Finished going through HVC-001
Parts:
- removed BC1, BC2: 0.1uF, symbol Device:C
- removed C1: 100uF, symbol Device:CP
- removed C10, C11, C12, C13, C15, C16, C17, C19, C3, C32, C4, C40: 0.01uF, symbol Device:C
- removed C2: 1N4148?, symbol Device:D
- removed C20, C21, C6: 220pF, symbol Device:C
- removed C27, C28, C29, C30, C31, C33, C34, C35, C36, C37, C5: 330pF, symbol Device:C
- removed C9: 2.2uF, symbol Device:CP
- removed DA1, DA3: DAN601, symbol _NTSCustom:DAN601
- removed DA2, DA4: uPA64H, symbol _NTSCustom:uPA64H
- removed FC1: 39uH, symbol Device:L
- removed FC2: ?uH, symbol Device:Ferrite_Bead
- removed P4: P1 PAD, symbol Connector:Conn_01x07_Male
- removed P5: P2 PAD, symbol Connector:Conn_01x07_Male
- removed P6: Power/Reset, symbol Connector:Conn_01x05_Male
- removed R1: 1M, symbol Device:R
- removed R14, R15: 5.6k, symbol Device:R
- removed R16: 10k, symbol Device:R
- removed R5: 220, symbol Device:R
- removed R6: 47K, symbol Device:R
- removed RA2: 6.8k, Resistor_THT:R_Array_SIP5, symbol Device:R_Network04
- removed RF_MOD1: RF MOD, symbol Connector:Conn_01x05_Male
- removed U10: 3193A, Package_DIP:DIP-16_W7.62mm, symbol _NTSCustom:3193A
- removed unit 1 of U9
- removed unit 3 of U9
- removed unit 4 of U9
- removed unit 5 of U9
- removed unit 6 of U9
- removed unit 2 of U9
- removed X2: 4MHz, symbol Device:Resonator
- added C1: 0.47uF, symbol Device:C
- added P1: CARTRIDGE, symbol Connector_Generic:Conn_02x30_Top_Bottom
- added P2: D-Jack, symbol Connector:DB15_Male
- added P3: RF Modulator, symbol Connector:Conn_01x07_Male
- added P4: P1 PAD, symbol Connector:Conn_01x05_Male
- added P5: P2 PAD, symbol Connector:Conn_01x06_Male
- added R12: 220, symbol Device:R
- added R7: 100K, symbol Device:R
- added R8: 10k, symbol Device:R
- added SW1: RESET, symbol Switch:SW_Push
- C18: value 0.01uF -> 68pF
- C7: value 220pF -> 0.1uF
- R3: renamed from R9; value 20K -> 10K
- R6: renamed from R2; value 510 -> 2.2K
- U7, U8: value 74LS368 -> TC40H368
- renumbered C46 to C11, C39 to C12, C25 to C13, C24 to C15, C22 to C16, C23 to C2, R3 to R1, R4 to R2, R7 to R4, R8 to R5, R4 to R9, RA1 to RM1
Connections:
- net PWR_LED is gone; now on net PPU_RD: C18.1
- net PWR_SW_IN is gone; now on net +5V: C14.1
- net RST_PB is gone; now on net GND: C8.2
- net +5V: now also U5.22 (~RST), P1.30 (Pin_30), P1.31 (Pin_31), P2.15 (P15), P3.2 (Pin_2), P3.3 (Pin_3), P3.4 (Pin_4), P4.5 (Pin_5), P5.6 (Pin_6); no longer C8.1
- net AUX_AUDIO_IN: no longer R3.2
- net AUX_VIDEO_OUT: no longer Q1.1 (E), R6.1
- net CIRAM_A10: now also P1.18 (Pin_18)
- net CIRAM_CE: now also P1.48 (Pin_48)
- net CPU_A0: now also P1.13 (Pin_13)
- net CPU_A1: now also P1.12 (Pin_12)
- net CPU_A10: now also P1.3 (Pin_3)
- net CPU_A11: now also P1.2 (Pin_2)
- net CPU_A12: now also P1.33 (Pin_33)
- net CPU_A13: now also P1.34 (Pin_34)
- net CPU_A14: now also P1.35 (Pin_35)
- net CPU_A2: now also P1.11 (Pin_11)
- net CPU_A3: now also P1.10 (Pin_10)
- net CPU_A4: now also P1.9 (Pin_9)
- net CPU_A5: now also P1.8 (Pin_8)
- net CPU_A6: now also P1.7 (Pin_7)
- net CPU_A7: now also P1.6 (Pin_6)
- net CPU_A8: now also P1.5 (Pin_5)
- net CPU_A9: now also P1.4 (Pin_4)
- net CPU_D0: now also U8.13 (O6b), P1.43 (Pin_43); no longer U8.3 (O1a)
- net CPU_D1: now also P1.42 (Pin_42)
- net CPU_D2: now also U8.11 (O5b), P1.41 (Pin_41); no longer U8.9 (O4a)
- net CPU_D3: now also U8.7 (O3a), P1.40 (Pin_40); no longer U7.11 (O5b), U8.11 (O5b)
- net CPU_D4: now also U8.9 (O4a), P1.39 (Pin_39); no longer U7.13 (O6b), U8.13 (O6b)
- net CPU_D5: now also P1.38 (Pin_38)
- net CPU_D6: now also P1.37 (Pin_37)
- net CPU_D7: now also P1.36 (Pin_36)
- net CPU_IRQ: now also RM1.2 (R1), P1.15 (Pin_15), P2.3; no longer RM1.7 (R6)
- net CPU_M2: now also U7.6 (I3), U8.2 (I1), P1.32 (Pin_32)
- net CPU_NMI: now also RM1.8 (R7); no longer RM1.13 (R12)
- net CPU_OE1: no longer U7.15 (OEb)
- net CPU_OUT0: now also P2.12 (P12), P4.3 (Pin_3), P5.4 (Pin_4)
- net CPU_OUT1: now also P2.11 (P111)
- net CPU_OUT2: now also P2.10 (P10)
- net CPU_RST: now also C1.1, SW1.2; no longer U5.22 (~RST)
- net CPU_RW: now also P1.14 (Pin_14)
- net GND: now also U7.15 (OEb), C1.2, P1.1 (Pin_1), P1.16 (Pin_16), P2.1, P3.1 (Pin_1), P3.6 (Pin_6), P4.1 (Pin_1), P5.2 (Pin_2), SW1.1; no longer U7.6 (I3), U8.6 (I3)
- net P1_D0: now also RM1.7 (R6), P4.2 (Pin_2); no longer RM1.9 (R8)
- net P1_D1: now also RM1.12 (R11), P2.13 (P13); no longer RM1.8 (R7)
- net P1_D2: no longer RM1.12 (R11), U7.10 (I4)
- net P1_D3: no longer RM1.10 (R9), U7.12 (I5)
- net P1_D4: no longer RM1.11 (R10), U7.14 (I6)
- net P2_D0: now also RM1.11 (R10), U8.14 (I6), P2.8, P5.3 (Pin_3); no longer RM1.3 (R2), U8.2 (I1)
- net P2_D1: now also RM1.10 (R9), P2.7; no longer RM1.2 (R1)
- net P2_D2: now also U8.12 (I5), P2.6; no longer U8.10 (I4)
- net P2_D3: now also U8.6 (I3), P2.5; no longer U8.12 (I5)
- net P2_D4: now also U8.10 (I4), P2.4; no longer U8.14 (I6)
- net PPU_!A13: now also U7.11 (O5b), P1.49 (Pin_49)
- net PPU_A0: now also U2.19 (O7), P1.25 (Pin_25); no longer U2.9 (O3)
- net PPU_A1: now also U2.16 (O6), P1.24 (Pin_24); no longer U2.12 (O4)
- net PPU_A10: now also P1.53 (Pin_53)
- net PPU_A11: now also P1.54 (Pin_54)
- net PPU_A12: now also P1.55 (Pin_55)
- net PPU_A13: now also U7.12 (I5), P1.56 (Pin_56)
- net PPU_A2: now also U2.15 (O5), P1.23 (Pin_23); no longer U2.6 (O2)
- net PPU_A3: now also U2.12 (O4), P1.22 (Pin_22); no longer U2.15 (O5)
- net PPU_A4: now also U2.9 (O3), P1.21 (Pin_21); no longer U2.5 (O1)
- net PPU_A5: now also U2.6 (O2), P1.20 (Pin_20); no longer U2.16 (O6)
- net PPU_A6: now also U2.5 (O1), P1.19 (Pin_19); no longer U2.2 (O0)
- net PPU_A7: now also U2.2 (O0), P1.50 (Pin_50); no longer U2.19 (O7)
- net PPU_A8: now also P1.51 (Pin_51)
- net PPU_A9: now also P1.52 (Pin_52)
- net PPU_AD0: now also U2.18 (D7), P1.26 (Pin_26); no longer U2.8 (D3)
- net PPU_AD1: now also U2.17 (D6), P1.27 (Pin_27); no longer U2.13 (D4)
- net PPU_AD2: now also U2.14 (D5), P1.28 (Pin_28); no longer U2.7 (D2)
- net PPU_AD3: now also U2.13 (D4), P1.29 (Pin_29); no longer U2.14 (D5)
- net PPU_AD4: now also U2.8 (D3), P1.60 (Pin_60); no longer U2.4 (D1)
- net PPU_AD5: now also U2.7 (D2), P1.59 (Pin_59); no longer U2.17 (D6)
- net PPU_AD6: now also U2.4 (D1), P1.58 (Pin_58); no longer U2.3 (D0)
- net PPU_AD7: now also U2.3 (D0), P1.57 (Pin_57); no longer U2.18 (D7)
- net PPU_RD: now also P1.17 (Pin_17)
- net PPU_WR: now also P1.47 (Pin_47)
- net ROMSEL: now also P1.44 (Pin_44)
- net VIDEO_OUT: now also P3.7 (Pin_7), R12.1
- net MIC_DIG_IN: now reaches C7.1
- net MIC_DIG_IN: now also U7.10 (I4), R8.1
- net TO_AF_AMP: now reaches C2.1
- net TO_AF_AMP: now also U7.14 (I6), R7.1
- net P1_M2: now reaches U7.7 (O3a)
- net P1_M2: now also RM1.13 (R12), P2.14 (P14), P4.4 (Pin_4)
- new net: Q1.1 (E), R12.2, R6.1
- new net AUDIO_TO_CART: C8.1, P1.45 (Pin_45), P2.2, R7.2, U7.13 (O6b)
- new net AUDIO_TO_RF_MOD: P1.46 (Pin_46), P3.5 (Pin_5)
- new net MIC_AUDIO_IN: P5.1 (Pin_1), R3.2, R8.2
- new net P2_M2: P2.9 (P9), P5.5 (Pin_5), RM1.3 (R2), U8.3 (O1a)
- no-connect marks 8 -> 6
Other:
- note added: "NES connectors for reference"
- note removed: "C6 and C7\nnot populated\n"
- note removed: "CIC\n"
- note removed: "Power/Reset Connector\n"
- note removed: "R14, R15, and R16\nnot populated\n"
- moved on the sheet: C15, C16, EDGE1, REFERENCE1, RM1, U3C, U7, U8, U9G
